File: EAGLE/finalSchematics.sch (EAGLE design)
At the start: 34 parts, among them IC1 STM32F103RBT, J2 U.FL, J3 U.FL, Q1 8MHz 131-220, U1 LM1117-3.3

Commit message: Death is near
Routing the board
Parts:
- added R1: 10k 901-655, rcl:R-EU_R0805
Connections:
- new net N$14: IC1.BOOT0, R1.2
- net +3V3: now also IC1.VBAT
- net GND: now also R1.1
Changed lines of the file:
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@@
 <part name="JP1" library="pinhead" deviceset="PINHD-1X3" device=""/>
 <part name="GND3" library="supply1" deviceset="GND" device=""/>
+<part name="R1" library="rcl" deviceset="R-EU_" device="R0805" value="10k 901-655"/>
+<part name="GND23" library="supply1" deviceset="GND" device=""/>
 </parts>
 <sheets>
@@
 <instance part="JP1" gate="A" x="187.96" y="137.16"/>
 <instance part="GND3" gate="1" x="177.8" y="121.92"/>
+<instance part="R1" gate="G$1" x="68.58" y="121.92" rot="R90"/>
+<instance part="GND23" gate="1" x="58.42" y="114.3" rot="R270"/>
 </instances>
 <busses>
@@
 <wire x1="177.8" y1="134.62" x2="177.8" y2="124.46" width="0.1524" layer="91"/>
 </segment>
+<segment>
+<pinref part="R1" gate="G$1" pin="1"/>
+<wire x1="68.58" y1="116.84" x2="68.58" y2="114.3" width="0.1524" layer="91"/>
+<pinref part="GND23" gate="1" pin="GND"/>
+<wire x1="68.58" y1="114.3" x2="60.96" y2="114.3" width="0.1524" layer="91"/>
+</segment>
 </net>
 <net name="CS-RAD" class="0">
@@
 <wire x1="71.12" y1="147.32" x2="71.12" y2="149.86" width="0.1524" layer="91"/>
 <junction x="71.12" y="149.86"/>
+<pinref part="IC1" gate="MCU" pin="VBAT"/>
+<wire x1="76.2" y1="152.4" x2="71.12" y2="152.4" width="0.1524" layer="91"/>
+<wire x1="71.12" y1="152.4" x2="71.12" y2="149.86" width="0.1524" layer="91"/>
 </segment>
 <segment>
@@
 </segment>
 </net>
+<net name="N$14" class="0">
+<segment>
+<pinref part="IC1" gate="MCU" pin="BOOT0"/>
+<wire x1="76.2" y1="132.08" x2="68.58" y2="132.08" width="0.1524" layer="91"/>
+<pinref part="R1" gate="G$1" pin="2"/>
+<wire x1="68.58" y1="132.08" x2="68.58" y2="127" width="0.1524" layer="91"/>
+</segment>
+</net>
 </nets>
 </sheet>
 </sheets>
+<errors>
+</errors>
 </schematic>
 </drawing>

Commit message: Finish Route PCB, prepare for inspection
Hakys je sport budoucnosti!
Parts:
- Q1: value 8MHz 131-220 -> (none); device crystal:CRYSTALHC49U-V -> crystal:CRYSTALHC49UP
Changed lines of the file:
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@@
 </classes>
 <parts>
-<part name="Q1" library="crystal" deviceset="CRYSTAL" device="HC49U-V" value="8MHz 131-220"/>
 <part name="C1" library="rcl" deviceset="C-EU" device="C0805" value="4.7p 906-099"/>
 <part name="C2" library="rcl" deviceset="C-EU" device="C0805" value="4.7p 906-099"/>
@@
 <part name="R1" library="rcl" deviceset="R-EU_" device="R0805" value="10k 901-655"/>
 <part name="GND23" library="supply1" deviceset="GND" device=""/>
+<part name="Q1" library="crystal" deviceset="CRYSTAL" device="HC49UP"/>
 </parts>
 <sheets>
@@
 </plain>
 <instances>
-<instance part="Q1" gate="G$1" x="66.04" y="161.29" smashed="yes" rot="R90">
-<attribute name="NAME" x="60.96" y="160.02" size="1.778" layer="95"/>
-<attribute name="VALUE" x="59.69" y="154.94" size="1.778" layer="96"/>
-</instance>
 <instance part="C1" gate="G$1" x="55.88" y="165.1" smashed="yes" rot="R90">
 <attribute name="NAME" x="52.324" y="166.751" size="1.778" layer="95"/>
@@
 <instance part="R1" gate="G$1" x="68.58" y="121.92" rot="R90"/>
 <instance part="GND23" gate="1" x="58.42" y="114.3" rot="R270"/>
+<instance part="Q1" gate="G$1" x="66.04" y="161.29" rot="R90"/>
 </instances>
 <busses>
@@
 <segment>
 <pinref part="C2" gate="G$1" pin="2"/>
-<pinref part="Q1" gate="G$1" pin="1"/>
 <wire x1="60.96" y1="157.48" x2="66.04" y2="157.48" width="0.1524" layer="91"/>
 <wire x1="66.04" y1="157.48" x2="66.04" y2="158.75" width="0.1524" layer="91"/>
@@
 <wire x1="71.12" y1="157.48" x2="71.12" y2="160.02" width="0.1524" layer="91"/>
 <wire x1="71.12" y1="160.02" x2="76.2" y2="160.02" width="0.1524" layer="91"/>
+<pinref part="Q1" gate="G$1" pin="1"/>
 </segment>
 </net>
 <net name="N$2" class="0">
 <segment>
-<pinref part="Q1" gate="G$1" pin="2"/>
 <pinref part="C1" gate="G$1" pin="2"/>
 <wire x1="66.04" y1="163.83" x2="66.04" y2="165.1" width="0.1524" layer="91"/>
@@
 <wire x1="71.12" y1="165.1" x2="66.04" y2="165.1" width="0.1524" layer="91"/>
 <junction x="66.04" y="165.1"/>
-</segment>
-</net>
+<pinref part="Q1" gate="G$1" pin="2"/>
+</segment>
+</net>

Commit message: Final fixes before etching
Parts:
- removed 1NF: (no value), rcl:C-EUC0805
- added C12: 1n, rcl:C-EUC0805
- C1, C2: value 4.7p 906-099 -> 15p
- C10, C11, C3, C6, C7, C8, C9: value (none) -> 100n
- J1: value (none) -> PWR
- JP1: value (none) -> DBG
- JP2: value (none) -> SWD
- LED1, LED2, LED3: value (none) -> GRN
- Q1: value (none) -> 8 MHz
- R4, R5, R6: value (none) -> 270
- SD1: value (none) -> SD
- renumbered 270OHM to R4, 270OHM1 to R6, 270OHM2 to R5
Connections:
- removed net N$4: D1.A, J1.1
- removed net N$8: 1NF.2, IC1.NRST
- net GND: now also C12.1, D1.A
- net N$3: now also J1.1
- net NRST: now also C12.2, IC1.NRST; no longer 1NF.1
Other:
- moved on the sheet: D1
